File: thermocouple-attiny1634.sch (KiCad schematic (older format))
At the start: 40 parts, among them CON1 AVR-ISP-6, IC1 SP3485CN, IC2 ATMEGA88-A, P1 CONN_2, P2 CONN_4, U1 AD8237, U2 TC1047, U3 7805, U4 LM358, X1 CRYSTAL

Commit message: visko daug
Parts:
- removed C17: 100nF, ~, symbol C
- removed IC2: ATMEGA88-A, TQFP32, symbol ATMEGA88-A
- added IC2: ATTINY1634-S, SO20, symbol ATTINY1634-S
Connections:
- wire segments 63 -> 58
Other:
- moved on the sheet: C13, C14, C15, C16, IC1, JP1, R8, R9, X1
